File: schematics/Battery.kicad_pcb (KiCad board)
At the start: 2 copper layers, 90 x 25 mm, 48 parts, among them J1 BATTERY, J2 CHG, J3 PWR, J4 3v3, J5 1v8, J6 NTC, Q1 Si9933CDY, U1 BQ29200, U2 LTC4002ES8, U3 MAX604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

Commit message: Update to KiCad 6
Other:
- net class Default removed
- board text added: "~{CHRG}"
- board text removed: "~CHRG"
