File: schematics/revision-2/Battery.kicad_pcb (KiCad board)
At the start: 2 copper layers, 90 x 25 mm, 48 parts, among them J1 BATTERY, J2 CHG, J3 PWR, J4 3v3, J5 1v8, J6 NTC, Q1 Si9933CDY, U1 BQ29200, U2 LTC4002ES8, U3 MAX604, U4 MAX604

Commit message: Fixes
Parts:
- removed C10, C11, C12, C9: 10u, Battery:C_0805_2012Metric_Pad1.18x1.45mm_HandSolder
- removed G***: LOGO, Battery:cusf_logo_full
- removed J4: 3v3, Battery:Molex_Nano-Fit_105313-xx02_1x02_P2.50mm_Horizontal
- removed J5: 1v8, Battery:Molex_Nano-Fit_105313-xx02_1x02_P2.50mm_Horizontal
- removed J6: NTC, Battery:Molex_Nano-Fit_105313-xx02_1x02_P2.50mm_Horizontal
- removed R8: 200k, Battery:R_0805_2012Metric_Pad1.20x1.40mm_HandSolder
- removed R9: 100k, Battery:R_0805_2012Metric_Pad1.20x1.40mm_HandSolder
- removed TP1, TP2, TP4, TP5, TP7, TP8: TestPoint, Battery:TestPoint_Pad_D2.0mm
- removed U3, U4: MAX604, Battery:SOIC-8_3.9x4.9mm_P1.27mm
- added D2: B330, Battery:D_SMB_Handsoldering, F.Cu at (119.0, 90.0)
- J1: footprint Battery:Molex_Nano-Fit_105313-xx03_1x03_P2.50mm_Horizontal -> Battery:SolderWire-0.25sqmm_1x03_P4.5mm_D0.65mm_OD2mm
- J2: footprint Battery:Molex_Nano-Fit_105313-xx02_1x02_P2.50mm_Horizontal -> Battery:SolderWire-0.25sqmm_1x02_P4.5mm_D0.65mm_OD2mm
- J3: value PWR -> SDN; footprint Battery:Molex_Nano-Fit_105313-xx02_1x02_P2.50mm_Horizontal -> Battery:SolderWire-0.25sqmm_1x02_P4.5mm_D0.65mm_OD2mm
- moved J1 82.8 mm to (197.0, 94.5), turned to -90 degrees
- moved J2 76.1 mm to (108.0, 96.0), turned to -90 degrees
- moved R2 62.2 mm to (183.0, 83.0)
- moved R3 61.5 mm to (183.0, 87.0)
- moved R4 58.3 mm to (183.0, 91.0), turned to 0 degrees
- moved U1 57.6 mm to (188.0, 99.0)
- moved C8 53.5 mm to (188.0, 108.0), turned to 0 degrees
- moved C2 52.7 mm to (180.0, 101.0), turned to 0 degrees
- moved C5 51.2 mm to (182.0, 107.0)
- moved C3 49.6 mm to (175.0, 106.0), turned to 0 degrees
- moved R6 48.5 mm to (183.0, 95.0), turned to 0 degrees
- moved TP10 44.7 mm to (166.3, 95.7)
- moved TP9 29.3 mm to (152.2, 111.2)
- moved R1 28.8 mm to (166.7, 92.1), turned to 0 degrees
- moved TP3 27.7 mm to (161.6, 102.7)
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Connections:
- J3 pad 1: VBATT -> Net-(C4-Pad1)
- U1 pad 9: (no net) -> GND
- U2 pad 8: Net-(J6-Pad1) -> GND
Routing:
- net GND: track 118.9 -> 0.00 mm, vias 40 -> 0
- net Net-(J2-Pad1): track 52.7 -> 0.00 mm, vias 2 -> 0
- net Net-(J6-Pad1): track 35.7 -> 0.00 mm, vias 2 -> 0
- net Net-(Q1-Pad4): track 26.3 -> 0.00 mm
- net /BATT_MON: track 25.8 -> 0.00 mm
- net Net-(C6-Pad1): track 23.8 -> 0.00 mm
- net Net-(D1-Pad1): track 22.6 -> 0.00 mm
- net 1v8: track 20.3 -> 0.00 mm
- net 3v3: track 16.9 -> 0.00 mm
- net Net-(Q1-Pad2): track 14.4 -> 0.00 mm
- net VBATT: track 7.78 -> 0.00 mm
- net Net-(TP3-Pad1): track 7.11 -> 0.00 mm
- net Net-(L1-Pad2): track 6.85 -> 0.00 mm
- net Net-(C2-Pad2): track 6.55 -> 0.00 mm
- net Net-(C2-Pad1): track 5.45 -> 0.00 mm
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- removed copper zone on B.Cu, net GND
- removed copper zone on F.Cu, net GND
- removed copper zone on F.Cu, net VBATT
Other:
- board outline removed
- board text removed: "1v8"
- board text removed: "2S Li-Ion Battery Charger H. E. Franks"
- board text removed: "3v3"
- board text removed: "CHG"
- board text removed: "GND"
- board text removed: "MON"
- board text removed: "NTC"
- board text removed: "OUT"
- board text removed: "V+"
- board text removed: "VBATT"
- board text removed: "VIN"
- board text removed: "~{CHRG}"

Commit message: Finish revision 2
Parts:
- removed R3: 261, Battery:R_0805_2012Metric_Pad1.20x1.40mm_HandSolder
- added G***: LOGO, Battery:cusf_logo_full, B.Cu at (162.0, 130.6)
- added GATE: TestPoint, Battery:TestPoint_Pad_D2.0mm, F.Cu at (174.9, 121.1)
- added R105: 100, Battery:R_0805_2012Metric_Pad1.20x1.40mm_HandSolder, F.Cu at (150.8, 129.4)
- added R106: 160, Battery:R_0805_2012Metric_Pad1.20x1.40mm_HandSolder, F.Cu at (147.5, 130.7)
- added SENSE: TestPoint, Battery:TestPoint_Pad_D2.0mm, F.Cu at (164.6, 126.8)
- added SW: TestPoint, Battery:TestPoint_Pad_D2.0mm, F.Cu at (168.0, 139.2)
- added VCC: TestPoint, Battery:TestPoint_Pad_D2.0mm, F.Cu at (185.0, 124.6)
- moved CHARGER 87.1 mm to (189.4, 127.0), turned to 90 degrees
- moved D101 77.2 mm to (184.6, 130.7), turned to -90 degrees
- moved Q101 68.8 mm to (179.2, 131.4), turned to -90 degrees
- moved BATTERY 62.7 mm to (143.6, 127.3)
- moved SHUTDOWN 62.5 mm to (189.4, 136.2), turned to -90 degrees
- moved C106 59.2 mm to (184.0, 137.2), turned to 180 degrees
- moved R107 52.1 mm to (150.8, 132.0)
- moved R104 50.7 mm to (155.8, 125.8), turned to -90 degrees
- moved D102 48.4 mm to (174.0, 132.8), turned to 90 degrees
- moved R108 46.5 mm to (184.0, 139.6)
- moved GND 45.3 mm to (143.6, 140.2)
- moved L101 45.1 mm to (167.8, 131.8), turned to 90 degrees
- moved U102 44.3 mm to (155.8, 129.5)
- moved MON 43.2 mm to (148.0, 134.8)
- moved R101 41.3 mm to (178.2, 137.0), turned to 90 degrees
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- renumbered TP9 to BATT, J1 to BATTERY, C6 to C101, C7 to C102, C2 to C103, C8 to C104, C3 to C105, C4 to C106, C1 to C107, C5 to C108, J2 to CHARGER, D2 to D101, D1 to D102, TP13 to GND, TP12 to GND, TP11 to GND, L1 to L101, TP10 to MON, TP3 to OUT, Q1 to Q101, R7 to R101, R6 to R102, R1 to R103, R2 to R104, R4 to R107, R5 to R108, J3 to SHUTDOWN, U2 to U101, U1 to U102, TP6 to ~{CHRG}
Connections:
- net Net-(C4-Pad1) renamed /COMP
- net Net-(C6-Pad1) renamed /VCC_CHG
- net Net-(D1-Pad1) renamed /V_SW
- net Net-(L1-Pad2) renamed /SENSE
- net Net-(Q1-Pad4) renamed /~{CHRG}
Routing:
- net /~{CHRG}: track 0.00 -> 24.2 mm, vias 0 -> 3
- net Net-(Q101-Pad2): track 0.00 -> 17.4 mm
- net /COMP: track 0.00 -> 16.8 mm, vias 0 -> 1
- net Net-(C103-Pad2): track 0.00 -> 7.39 mm
- net Net-(TP106-Pad1): track 0.00 -> 5.02 mm
- net GND: track 0.00 -> 4.75 mm, vias 0 -> 3
- net Net-(C103-Pad1): track 0.00 -> 4.16 mm
- net Net-(C104-Pad1): track 0.00 -> 3.94 mm
- net Net-(R107-Pad2): track 0.00 -> 3.70 mm
- net /SENSE: track 0.00 -> 2.78 mm
- net VBATT: track 0.00 -> 2.78 mm
- net Net-(R105-Pad1): track 0.00 -> 2.42 mm
- net Net-(C106-Pad2): track 0.00 -> 2.42 mm
- net Net-(C108-Pad1): track 0.00 -> 1.97 mm
- added copper zone on F.Cu, net /BATT_MON
- added copper zone on F.Cu, net /COMP
- added copper zone on F.Cu, net /SENSE
- added copper zone on F.Cu, net /VCC_CHG
- added copper zone on F.Cu, net /V_SW
- added copper zone on B.Cu, net GND
- added copper zone on F.Cu, net GND
- added copper zone on F.Cu, net Net-(D101-Pad2)
- added copper zone on F.Cu, net VBATT
Other:
- board outline added: 52.8 x 25.6 mm
- board text added: "Designed by H. Franks Jan. 2022"
- board text added: "Li-Ion Battery Charger v2"
