File: schematics/revision-2/Battery.kicad_sch (KiCad schematic)
At the start: 31 parts, among them J1 BATTERY, J2 CHG, J3 SDN, Q1 Si9933CDY, U1 BQ29200, U2 LTC4002ES8

Commit message: Fixes
Parts:
- gave numbers to parts that had none: 1
Connections:
- net GND: now also U1.9 (PGND)
Other:
- moved on the sheet: TP10, TP11, TP12, TP13, TP9

Commit message: Finish revision 2
Parts:
- removed R3: 261, Battery:R_0805_2012Metric_Pad1.20x1.40mm_HandSolder, symbol Battery:R
- added R105: 100, Battery:R_0805_2012Metric_Pad1.20x1.40mm_HandSolder, symbol Battery:R
- added R106: 160, Battery:R_0805_2012Metric_Pad1.20x1.40mm_HandSolder, symbol Battery:R
- added TP101, TP102, TP103, TP105: TestPoint, Battery:TestPoint_Pad_D2.0mm, symbol Battery:TestPoint
- renumbered C6 to C101, C7 to C102, C2 to C103, C8 to C104, C3 to C105, C4 to C106, C1 to C107, C5 to C108, D2 to D101, D1 to D102, J2 to J101, J1 to J102, J3 to J103, L1 to L101, Q1 to Q101, R7 to R101, R6 to R102, R1 to R103, R2 to R104, R4 to R107, R5 to R108, TP6 to TP104, TP3 to TP106, TP9 to TP107, TP10 to TP108, TP11 to TP109, TP12 to TP110, TP13 to TP111, U2 to U101, U1 to U102
Connections:
- net BATT_MON: now also R106.1
- net at C103.2, C105.1, U102.2 (VC1): now also R105.2
- net COMP: now reaches C106.1, J103.1 (Pin_1), U101.1 (COMP)
- net VCC_CHG: now reaches C101.1, C102.1, D101.1, Q101.1 (S1), Q101.3 (S2), U101.2 (VCC)
- net VCC_CHG: now also TP101.1
- net at Q101.2 (G1), U101.3 (GATE): now also TP102.1
- net ~{CHRG}: now reaches Q101.4 (G2), R101.1, TP104.1, U101.5 (~{CHRG})
- net SENSE: now reaches L101.2, R103.2, U101.7 (SENSE)
- net SENSE: now also TP105.1
- net V_SW: now reaches D102.1, L101.1, Q101.7 (D1), Q101.8 (D1)
- net V_SW: now also TP103.1
- new net: R105.1, R106.2
Other:
- moved on the sheet: R104, R107
